File: InputKeys.sch (KiCad schematic (older format))
At the start: 52 parts, among them SW101 TL-1240-NO_LED, SW102 TL-1240-NO_LED, SW103 TL-1240-NO_LED, SW104 TL-1240-NO_LED, SW105 TL-1240-NO_LED, SW106 TL-1240-NO_LED, SW107 TL-1240-NO_LED, SW108 TL-1240-NO_LED, SW109 TL-1240-NO_LED, SW110 TL-1240-NO_LED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

Commit message: Add JLCPCB assembly stuff, update plots
Parts:
- C101, C102, C103, C104, C105, C106, C107, C108, C109, C110, C111, C112: JLC (none) -> 0603; LCSC (none) -> C115056
- C113, C114: JLC (none) -> 0603; LCSC (none) -> C14663
- R101, R102, R103, R104, R105, R106, R107, R108, R109, R110, R111, R112, R113, R114, R115, R116, R117, R118, R119, R120, R121, R122, R123, R124: JLC (none) -> 0603; LCSC (none) -> C98220
- U101, U102: JLC (none) -> TSSOP-14; LCSC (none) -> C6066
