File: MCU_LAN.sch (KiCad schematic (older format))
At the start: 5 parts, among them J301 ENC28J60, SW301 SW_ForceSetup, SW302 SW_Reset, SW303 OS102011MA1QN1C, U301 DOIT-ESP32-DEVKIT-V1_30PIN

Commit message: Add JLCPCB assembly stuff, update plots
Parts:
- SW301, SW302: JLC (none) -> SMD; LCSC (none) -> C388883
Changed lines of the file:
@@
 F 2 "Button_Switch_SMD:SW_SPST_EVQP7C" H 3150 6250 50  0001 C CNN
 F 3 "~" H 3150 6250 50  0001 C CNN
+F 4 "SMD" H 3150 6050 50  0001 C CNN "JLC"
+F 5 "C388883" H 3150 6050 50  0001 C CNN "LCSC"
 	1    3150 6050
 	1    0    0    -1
@@
 F 2 "Button_Switch_SMD:SW_SPST_EVQP7C" H 3150 6700 50  0001 C CNN
 F 3 "~" H 3150 6700 50  0001 C CNN
+F 4 "SMD" H 3150 6500 50  0001 C CNN "JLC"
+F 5 "C388883" H 3150 6500 50  0001 C CNN "LCSC"
 	1    3150 6500
 	1    0    0    -1
