File: Navigation_Power.sch (KiCad schematic (older format))
At the start: 22 parts, among them SW201 TL-1240-NO_LED, SW202 TL-1240-NO_LED, SW203 TL-1240-NO_LED, SW204 TL-1240-NO_LED, SW205 TL-1240-NO_LED, U201 74HC14

Commit message: Add JLCPCB assembly stuff, update plots
Parts:
- C201, C202, C203, C204, C205: JLC (none) -> 0603; LCSC (none) -> C115056
- C206: JLC (none) -> 0603; LCSC (none) -> C14663
- R201, R202, R203, R204, R205, R206, R207, R208, R209, R210: JLC (none) -> 0603; LCSC (none) -> C98220
- U201: JLC (none) -> TSSOP-14; LCSC (none) -> C6066
Changed lines of the file:
@@
 F 2 "Resistor_SMD:R_0603_1608Metric_Pad0.98x0.95mm_HandSolder" H 1600 1350 50  0001 C CNN
 F 3 "~" H 1600 1350 50  0001 C CNN
+F 4 "0603" H 1600 1350 50  0001 C CNN "JLC"
+F 5 "C98220" H 1600 1350 50  0001 C CNN "LCSC"
 	1    1600 1350
 	1    0    0    -1
@@
 F 2 "Resistor_SMD:R_0603_1608Metric_Pad0.98x0.95mm_HandSolder" H 2800 1550 50  0001 C CNN
 F 3 "~" H 2800 1550 50  0001 C CNN
+F 4 "0603" H 2800 1550 50  0001 C CNN "JLC"
+F 5 "C98220" H 2800 1550 50  0001 C CNN "LCSC"
 	1    2800 1550
 	0    1    1    0
@@
 F 2 "Capacitor_SMD:C_0603_1608Metric_Pad1.08x0.95mm_HandSolder" H 3000 1750 50  0001 C CNN
 F 3 "~" H 3000 1750 50  0001 C CNN
+F 4 "0603" H 3000 1750 50  0001 C CNN "JLC"
+F 5 "C115056" H 3000 1750 50  0001 C CNN "LCSC"
 	1    3000 1750
 	1    0    0    -1
@@
 F 2 "Package_SO:TSSOP-14_4.4x5mm_P0.65mm" H 3400 1550 50  0001 C CNN
 F 3 "http://www.ti.com/lit/gpn/sn74HC14" H 3400 1550 50  0001 C CNN
+F 4 "TSSOP-14" H 3400 1550 50  0001 C CNN "JLC"
+F 5 "C6066" H 3400 1550 50  0001 C CNN "LCSC"
 	1    3400 1550
 	1    0    0    -1
@@
 F 2 "Resistor_SMD:R_0603_1608Metric_Pad0.98x0.95mm_HandSolder" H 5000 1400 50  0001 C CNN
 F 3 "~" H 5000 1400 50  0001 C CNN
+F 4 "0603" H 5000 1400 50  0001 C CNN "JLC"
+F 5 "C98220" H 5000 1400 50  0001 C CNN "LCSC"
 	1    5000 1400
 	1    0    0    -1
@@
 F 2 "Resistor_SMD:R_0603_1608Metric_Pad0.98x0.95mm_HandSolder" H 6200 1600 50  0001 C CNN
 F 3 "~" H 6200 1600 50  0001 C CNN
+F 4 "0603" H 6200 1600 50  0001 C CNN "JLC"
+F 5 "C98220" H 6200 1600 50  0001 C CNN "LCSC"
 	1    6200 1600
 	0    1    1    0
@@
 F 2 "Capacitor_SMD:C_0603_1608Metric_Pad1.08x0.95mm_HandSolder" H 6400 1800 50  0001 C CNN
 F 3 "~" H 6400 1800 50  0001 C CNN
+F 4 "0603" H 6400 1800 50  0001 C CNN "JLC"
+F 5 "C115056" H 6400 1800 50  0001 C CNN "LCSC"
 	1    6400 1800
 	1    0    0    -1
@@
 F 2 "Package_SO:TSSOP-14_4.4x5mm_P0.65mm" H 6800 1600 50  0001 C CNN
 F 3 "http://www.ti.com/lit/gpn/sn74HC14" H 6800 1600 50  0001 C CNN
+F 4 "TSSOP-14" H 6800 1600 50  0001 C CNN "JLC"
+F 5 "C6066" H 6800 1600 50  0001 C CNN "LCSC"
 	2    6800 1600
 	1    0    0    -1
@@
 F 2 "Resistor_SMD:R_0603_1608Metric_Pad0.98x0.95mm_HandSolder" H 1600 2850 50  0001 C CNN
 F 3 "~" H 1600 2850 50  0001 C CNN
+F 4 "0603" H 1600 2850 50  0001 C CNN "JLC"
+F 5 "C98220" H 1600 2850 50  0001 C CNN "LCSC"
 	1    1600 2850
 	1    0    0    -1
@@
 F 2 "Resistor_SMD:R_0603_1608Metric_Pad0.98x0.95mm_HandSolder" H 2800 3050 50  0001 C CNN
 F 3 "~" H 2800 3050 50  0001 C CNN
+F 4 "0603" H 2800 3050 50  0001 C CNN "JLC"
+F 5 "C98220" H 2800 3050 50  0001 C CNN "LCSC"
 	1    2800 3050
 	0    1    1    0
@@
 F 2 "Capacitor_SMD:C_0603_1608Metric_Pad1.08x0.95mm_HandSolder" H 3000 3250 50  0001 C CNN
 F 3 "~" H 3000 3250 50  0001 C CNN
+F 4 "0603" H 3000 3250 50  0001 C CNN "JLC"
+F 5 "C115056" H 3000 3250 50  0001 C CNN "LCSC"
 	1    3000 3250
 	1    0    0    -1
@@
 F 2 "Package_SO:TSSOP-14_4.4x5mm_P0.65mm" H 3450 5350 50  0001 C CNN
 F 3 "http://www.ti.com/lit/gpn/sn74HC14" H 3450 5350 50  0001 C CNN
+F 4 "TSSOP-14" H 3450 5350 50  0001 C CNN "JLC"
+F 5 "C6066" H 3450 5350 50  0001 C CNN "LCSC"
 	3    3450 5350
 	1    0    0    -1
@@
 F 2 "Resistor_SMD:R_0603_1608Metric_Pad0.98x0.95mm_HandSolder" H 5000 2900 50  0001 C CNN
 F 3 "~" H 5000 2900 50  0001 C CNN
+F 4 "0603" H 5000 2900 50  0001 C CNN "JLC"
+F 5 "C98220" H 5000 2900 50  0001 C CNN "LCSC"
 	1    5000 2900
 	1    0    0    -1
@@
 F 2 "Resistor_SMD:R_0603_1608Metric_Pad0.98x0.95mm_HandSolder" H 6200 3100 50  0001 C CNN
 F 3 "~" H 6200 3100 50  0001 C CNN
+F 4 "0603" H 6200 3100 50  0001 C CNN "JLC"
+F 5 "C98220" H 6200 3100 50  0001 C CNN "LCSC"
 	1    6200 3100
 	0    1    1    0
@@
 F 2 "Capacitor_SMD:C_0603_1608Metric_Pad1.08x0.95mm_HandSolder" H 6400 3300 50  0001 C CNN
 F 3 "~" H 6400 3300 50  0001 C CNN
+F 4 "0603" H 6400 3300 50  0001 C CNN "JLC"
+F 5 "C115056" H 6400 3300 50  0001 C CNN "LCSC"
 	1    6400 3300
 	1    0    0    -1
@@
 F 2 "Package_SO:TSSOP-14_4.4x5mm_P0.65mm" H 6800 3100 50  0001 C CNN
 F 3 "http://www.ti.com/lit/gpn/sn74HC14" H 6800 3100 50  0001 C CNN
+F 4 "TSSOP-14" H 6800 3100 50  0001 C CNN "JLC"
+F 5 "C6066" H 6800 3100 50  0001 C CNN "LCSC"
 	4    6800 3100
 	1    0    0    -1
@@
 F 2 "Resistor_SMD:R_0603_1608Metric_Pad0.98x0.95mm_HandSolder" H 1650 5150 50  0001 C CNN
 F 3 "~" H 1650 5150 50  0001 C CNN
+F 4 "0603" H 1650 5150 50  0001 C CNN "JLC"
+F 5 "C98220" H 1650 5150 50  0001 C CNN "LCSC"
 	1    1650 5150
 	1    0    0    -1
@@
 F 2 "Resistor_SMD:R_0603_1608Metric_Pad0.98x0.95mm_HandSolder" H 2850 5350 50  0001 C CNN
 F 3 "~" H 2850 5350 50  0001 C CNN
+F 4 "0603" H 2850 5350 50  0001 C CNN "JLC"
+F 5 "C98220" H 2850 5350 50  0001 C CNN "LCSC"
 	1    2850 5350
 	0    1    1    0
@@
 F 2 "Capacitor_SMD:C_0603_1608Metric_Pad1.08x0.95mm_HandSolder" H 3050 5550 50  0001 C CNN
 F 3 "~" H 3050 5550 50  0001 C CNN
+F 4 "0603" H 3050 5550 50  0001 C CNN "JLC"
+F 5 "C115056" H 3050 5550 50  0001 C CNN "LCSC"
 	1    3050 5550
 	1    0    0    -1
@@
 F 2 "Package_SO:TSSOP-14_4.4x5mm_P0.65mm" H 3400 3050 50  0001 C CNN
 F 3 "http://www.ti.com/lit/gpn/sn74HC14" H 3400 3050 50  0001 C CNN
+F 4 "TSSOP-14" H 3400 3050 50  0001 C CNN "JLC"
+F 5 "C6066" H 3400 3050 50  0001 C CNN "LCSC"
 	5    3400 3050
 	1    0    0    -1
@@
 F 2 "Package_SO:TSSOP-14_4.4x5mm_P0.65mm" H 5850 5350 50  0001 C CNN
 F 3 "http://www.ti.com/lit/gpn/sn74HC14" H 5850 5350 50  0001 C CNN
+F 4 "TSSOP-14" H 5850 5350 50  0001 C CNN "JLC"
+F 5 "C6066" H 5850 5350 50  0001 C CNN "LCSC"
 	6    5850 5350
 	1    0    0    -1
@@
 F 2 "Package_SO:TSSOP-14_4.4x5mm_P0.65mm" H 2000 6950 50  0001 C CNN
 F 3 "http://www.ti.com/lit/gpn/sn74HC14" H 2000 6950 50  0001 C CNN
+F 4 "TSSOP-14" H 2000 6950 50  0001 C CNN "JLC"
+F 5 "C6066" H 2000 6950 50  0001 C CNN "LCSC"
 	7    2000 6950
 	1    0    0    -1
@@
 F 2 "Capacitor_SMD:C_0603_1608Metric_Pad1.08x0.95mm_HandSolder" H 2200 6400 50  0001 C CNN
 F 3 "~" H 2200 6400 50  0001 C CNN
+F 4 "0603" H 2200 6400 50  0001 C CNN "JLC"
+F 5 "C14663" H 2200 6400 50  0001 C CNN "LCSC"
 	1    2200 6400
 	0    1    1    0
