File: bkm-15r-mini.kicad_pcb (KiCad board)
At the start: 2 copper layers, 91 x 57 mm, 84 parts, among them J301 ENC28J60, SW101 TL-1240-NO_LED, SW102 TL-1240-NO_LED, SW103 TL-1240-NO_LED, SW104 TL-1240-NO_LED, SW105 TL-1240-NO_LED, SW106 TL-1240-NO_LED, SW107 TL-1240-NO_LED, SW108 TL-1240-NO_LED, SW109 TL-1240-NO_LED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

Commit message: Add JLCPCB assembly stuff, update plots
Parts:
- SW303: value SW_SPDT -> OS102011MA1QN1C
